File: HW/V1/V1.kicad_pcb (KiCad board)
At the start: 2 copper layers, 8 parts, among them J3 WellerConn, U2 OLED_128x64_i2c_0.96

Commit message: Fized bugs
Parts:
- added Q1: Si4435, Package_SO:SOIC-8_3.9x4.9mm_P1.27mm, B.Cu at (106.0, 100.9)
Connections:
- J3 pad 5: Net-(J3-Pad5) -> HandleTempRaw
- J3 pad 6: HandleTempRaw -> Net-(J3-Pad6)
