File: HW/V2/Power.sch (KiCad schematic (older format))
At the start: 17 parts, among them J2 +24VDC, J4 +7.5VDC, U1 MAX6126_50, U2 AP2210-3.3V, U4 DS2401Z

Commit message: V2 milling and BOM
Parts:
- removed J2: +24VDC, TerminalBlock_MetzConnect:TerminalBlock_MetzConnect_Type175_RT02702HBLC_1x02_P7.50mm_Horizontal, symbol Connector:Screw_Terminal_01x02
- removed J4: +7.5VDC, TerminalBlock:TerminalBlock_bornier-2_P5.08mm, symbol Connector:Screw_Terminal_01x02
- removed R20: 1K5-5K, Resistor_SMD:R_0805_2012Metric_Pad1.15x1.40mm_HandSolder, symbol Device:R
- removed TP1: VrefTest, TestPoint:TestPoint_Loop_D2.50mm_Drill1.0mm, symbol Connector:TestPoint
- removed U4: DS2401Z, Package_TO_SOT_SMD:SOT-223, symbol Memory_UniqueID:DS2401Z
- added C6: 68uf, Capacitor_SMD:C_1210_3225Metric_Pad1.42x2.65mm_HandSolder, symbol Device:C
- added U15: +7.5VDC, Libs:Conn_Microfit_Vertical_molex, symbol Peters:Micro_MATE-N-LOK_3-794633-4_4PinMolex
- added U7: +24VDC, Libs:Conn_Microfit_Vertical_molex, symbol Peters:Micro_MATE-N-LOK_3-794633-4_4PinMolex
- C1: value 68uf -> 100N; footprint Capacitor_SMD:C_1210_3225Metric_Pad1.42x2.65mm_HandSolder -> Capacitor_SMD:C_0805_2012Metric_Pad1.15x1.40mm_HandSolder
Connections:
- net labels removed: oneWireTemp
- wire segments 47 -> 51
Changed lines of the file:
@@
 $EndComp
-$Comp
-L Device:C_Small C1
-U 1 1 5C631055
-P 1150 7050
-F 0 "C1" H 1242 7096 50  0000 L CNN
-F 1 "68uf" H 1242 7005 50  0000 L CNN
-F 2 "Capacitor_SMD:C_1210_3225Metric_Pad1.42x2.65mm_HandSolder" H 1150 7050 50  0001 C CNN
-F 3 "~" H 1150 7050 50  0001 C CNN
-	1    1150 7050
-	1    0    0    -1
-$EndComp
-Wire Wire Line
-	1550 6950 1150 6950
-Connection ~ 1550 6950
-Wire Wire Line
-	1550 7200 1150 7200
-Wire Wire Line
-	1150 7200 1150 7150
-Connection ~ 1550 7200
 $Comp
 L Peters:AP2210-3.3V U2
@@
 	1    0    0    -1
 $EndComp
-$Comp
-L Connector:TestPoint TP1
-U 1 1 5C738707
-P 3500 7050
-F 0 "TP1" H 3558 7170 50  0000 L CNN
-F 1 "VrefTest" H 3558 7079 50  0000 L CNN
-F 2 "TestPoint:TestPoint_Loop_D2.50mm_Drill1.0mm" H 3700 7050 50  0001 C CNN
-F 3 "~" H 3700 7050 50  0001 C CNN
-	1    3500 7050
-	1    0    0    -1
-$EndComp
-Wire Wire Line
-	3500 7050 3150 7050
-$Comp
-L Memory_UniqueID:DS2401Z U4
-U 1 1 5C6B6326
-P 5350 4450
-F 0 "U4" H 5579 4496 50  0000 L CNN
-F 1 "DS2401Z" H 5579 4405 50  0000 L CNN
-F 2 "Package_TO_SOT_SMD:SOT-223" H 5200 4700 50  0001 C CNN
-F 3 "http://pdfserv.maximintegrated.com/en/ds/DS2401.pdf" H 5200 4700 50  0001 C CNN
-	1    5350 4450
-	1    0    0    -1
-$EndComp
-$Comp
-L Device:R R20
-U 1 1 5C6B632D
-P 4850 4100
-F 0 "R20" H 4920 4146 50  0000 L CNN
-F 1 "1K5-5K" H 4920 4055 50  0000 L CNN
-F 2 "Resistor_SMD:R_0805_2012Metric_Pad1.15x1.40mm_HandSolder" V 4780 4100 50  0001 C CNN
-F 3 "~" H 4850 4100 50  0001 C CNN
-	1    4850 4100
-	1    0    0    -1
-$EndComp
-$Comp
-L power:VCC #PWR0130
-U 1 1 5C6B6334
-P 4850 3900
-F 0 "#PWR0130" H 4850 3750 50  0001 C CNN
-F 1 "VCC" H 4867 4073 50  0000 C CNN
-F 2 "" H 4850 3900 50  0001 C CNN
-F 3 "" H 4850 3900 50  0001 C CNN
-	1    4850 3900
-	1    0    0    -1
-$EndComp
-Text HLabel 4850 4350 0    50   Input ~ 0
-oneWireTemp
-Wire Wire Line
-	4850 3950 4850 3900
-$Comp
-L power:GND #PWR0131
-U 1 1 5C6B633C
-P 4950 4700
-F 0 "#PWR0131" H 4950 4450 50  0001 C CNN
-F 1 "GND" H 4955 4527 50  0000 C CNN
-F 2 "" H 4950 4700 50  0001 C CNN
-F 3 "" H 4950 4700 50  0001 C CNN
-	1    4950 4700
-	1    0    0    -1
-$EndComp
-Wire Wire Line
-	5050 4550 4950 4550
-Wire Wire Line
-	4950 4550 4950 4700
-Wire Wire Line
-	5050 4450 4850 4450
-Wire Wire Line
-	4850 4250 4850 4450
-Wire Wire Line
-	5050 4350 4950 4350
-Wire Wire Line
-	4950 4350 4950 4550
-Connection ~ 4950 4550
 Text GLabel 3150 6900 1    50   Input ~ 0
 +5vREF
 $Comp
-L Connector:Screw_Terminal_01x02 J2
-U 1 1 5C631334
-P 2650 1850
-F 0 "J2" H 2729 1842 50  0000 L CNN
-F 1 "+24VDC" H 2729 1751 50  0000 L CNN
-F 2 "TerminalBlock_MetzConnect:TerminalBlock_MetzConnect_Type175_RT02702HBLC_1x02_P7.50mm_Horizontal" H 2650 1850 50  0001 C CNN
-F 3 "~" H 2650 1850 50  0001 C CNN
-	1    2650 1850
-	-1   0    0    1
-$EndComp
-$Comp
-L Connector:Screw_Terminal_01x02 J4
-U 1 1 5C6313E4
-P 2700 1250
-F 0 "J4" H 2779 1242 50  0000 L CNN
-F 1 "+7.5VDC" H 2779 1151 50  0000 L CNN
-F 2 "TerminalBlock:TerminalBlock_bornier-2_P5.08mm" H 2700 1250 50  0001 C CNN
-F 3 "~" H 2700 1250 50  0001 C CNN
-	1    2700 1250
-	-1   0    0    1
-$EndComp
-$Comp
 L power:GND #PWR0118
 U 1 1 5C63148C
-P 2850 1900
-F 0 "#PWR0118" H 2850 1650 50  0001 C CNN
-F 1 "GND" H 2855 1727 50  0000 C CNN
-F 2 "" H 2850 1900 50  0001 C CNN
-F 3 "" H 2850 1900 50  0001 C CNN
-	1    2850 1900
-	1    0    0    -1
-$EndComp
-Wire Wire Line
-	2850 1900 2850 1850
+P 2000 2550
+F 0 "#PWR0118" H 2000 2300 50  0001 C CNN
+F 1 "GND" H 2005 2377 50  0000 C CNN
+F 2 "" H 2000 2550 50  0001 C CNN
+F 3 "" H 2000 2550 50  0001 C CNN
+	1    2000 2550
+	1    0    0    -1
+$EndComp
 $Comp
 L power:GND #PWR0120
 U 1 1 5C634A01
-P 2900 1250
-F 0 "#PWR0120" H 2900 1000 50  0001 C CNN
-F 1 "GND" H 2905 1077 50  0000 C CNN
-F 2 "" H 2900 1250 50  0001 C CNN
-F 3 "" H 2900 1250 50  0001 C CNN
-	1    2900 1250
+P 2650 1600
+F 0 "#PWR0120" H 2650 1350 50  0001 C CNN
+F 1 "GND" H 2655 1427 50  0000 C CNN
+F 2 "" H 2650 1600 50  0001 C CNN
+F 3 "" H 2650 1600 50  0001 C CNN
+	1    2650 1600
 	1    0    0    -1
 $EndComp
@@
 L power:+7.5V #PWR0121
 U 1 1 5C634AE9
-P 2900 1150
-F 0 "#PWR0121" H 2900 1000 50  0001 C CNN
-F 1 "+7.5V" H 2915 1323 50  0000 C CNN
-F 2 "" H 2900 1150 50  0001 C CNN
-F 3 "" H 2900 1150 50  0001 C CNN
-	1    2900 1150
+P 2650 1100
+F 0 "#PWR0121" H 2650 950 50  0001 C CNN
+F 1 "+7.5V" H 2665 1273 50  0000 C CNN
+F 2 "" H 2650 1100 50  0001 C CNN
+F 3 "" H 2650 1100 50  0001 C CNN
+	1    2650 1100
 	1    0    0    -1
 $EndComp
@@
 L power:+24V #PWR0122
 U 1 1 5C634C07
-P 2850 1700
-F 0 "#PWR0122" H 2850 1550 50  0001 C CNN
-F 1 "+24V" H 2865 1873 50  0000 C CNN
-F 2 "" H 2850 1700 50  0001 C CNN
-F 3 "" H 2850 1700 50  0001 C CNN
-	1    2850 1700
-	1    0    0    -1
-$EndComp
-Wire Wire Line
-	2850 1700 2850 1750
+P 1300 2200
+F 0 "#PWR0122" H 1300 2050 50  0001 C CNN
+F 1 "+24V" H 1315 2373 50  0000 C CNN
+F 2 "" H 1300 2200 50  0001 C CNN
+F 3 "" H 1300 2200 50  0001 C CNN
+	1    1300 2200
+	1    0    0    -1
+$EndComp
+Wire Wire Line
+	1300 2200 1300 2250
+$Comp
+L Device:C C6
+U 1 1 5C616B10
+P 2650 1350
+F 0 "C6" H 2765 1396 50  0000 L CNN
+F 1 "68uf" H 2765 1305 50  0000 L CNN
+F 2 "Capacitor_SMD:C_1210_3225Metric_Pad1.42x2.65mm_HandSolder" H 2688 1200 50  0001 C CNN
+F 3 "~" H 2650 1350 50  0001 C CNN
+	1    2650 1350
+	1    0    0    -1
+$EndComp
+Wire Wire Line
+	2650 1600 2650 1550
+Wire Wire Line
+	2650 1100 2650 1150
+$Comp
+L Peters:Micro_MATE-N-LOK_3-794633-4_4PinMolex U7
+U 1 1 5C61B357
+P 1650 2350
+F 0 "U7" H 1650 2765 50  0000 C CNN
+F 1 "+24VDC" H 1650 2674 50  0000 C CNN
+F 2 "Libs:Conn_Microfit_Vertical_molex" H 1600 2700 50  0001 C CNN
+F 3 "http://192.168.0.102/api/part_attachments/287/getFile" H 1100 2800 50  0001 C CNN
+	1    1650 2350
+	-1   0    0    1
+$EndComp
+$Comp
+L Peters:Micro_MATE-N-LOK_3-794633-4_4PinMolex U15
+U 1 1 5C61B3C4
+P 1850 1250
+F 0 "U15" H 1850 1665 50  0000 C CNN
+F 1 "+7.5VDC" H 1850 1574 50  0000 C CNN
+F 2 "Libs:Conn_Microfit_Vertical_molex" H 1800 1600 50  0001 C CNN
+F 3 "http://192.168.0.102/api/part_attachments/287/getFile" H 1300 1700 50  0001 C CNN
+	1    1850 1250
+	-1   0    0    1
+$EndComp
+$Comp
+L power:+24V #PWR0123
+U 1 1 5C61BEF0
+P 2000 2250
+F 0 "#PWR0123" H 2000 2100 50  0001 C CNN
+F 1 "+24V" H 2015 2423 50  0000 C CNN
+F 2 "" H 2000 2250 50  0001 C CNN
+F 3 "" H 2000 2250 50  0001 C CNN
+	1    2000 2250
+	1    0    0    -1
+$EndComp
+$Comp
+L power:GND #PWR0124
+U 1 1 5C61C963
+P 1300 2500
+F 0 "#PWR0124" H 1300 2250 50  0001 C CNN
+F 1 "GND" H 1305 2327 50  0000 C CNN
+F 2 "" H 1300 2500 50  0001 C CNN
+F 3 "" H 1300 2500 50  0001 C CNN
+	1    1300 2500
+	1    0    0    -1
+$EndComp
+Wire Wire Line
+	1300 2450 1300 2500
+Wire Wire Line
+	2200 1150 2350 1150
+Wire Wire Line
+	1500 1150 1500 800
+Wire Wire Line
+	1500 800  2350 800
+Wire Wire Line
+	2350 800  2350 1150
+Wire Wire Line
+	1500 1350 1500 1600
+Wire Wire Line
+	2200 1550 2650 1550
+Connection ~ 2650 1550
+Wire Wire Line
+	2650 1550 2650 1500
+Wire Wire Line
+	1500 1600 2200 1600
+Wire Wire Line
+	2200 1600 2200 1550
+Connection ~ 2200 1550
+Wire Wire Line
+	2650 1150 2350 1150
+Connection ~ 2650 1150
+Wire Wire Line
+	2650 1150 2650 1200
+Connection ~ 2350 1150
+Wire Wire Line
+	2000 2450 2000 2550
+Wire Wire Line
+	2200 1350 2200 1550
+$Comp
+L Device:C_Small C1
+U 1 1 5C618AC4
+P 2000 6650
+F 0 "C1" H 2092 6696 50  0000 L CNN
+F 1 "100N" H 2092 6605 50  0000 L CNN
+F 2 "Capacitor_SMD:C_0805_2012Metric_Pad1.15x1.40mm_HandSolder" H 2000 6650 50  0001 C CNN
+F 3 "~" H 2000 6650 50  0001 C CNN
+	1    2000 6650
+	1    0    0    -1
+$EndComp
+$Comp
+L power:GND #PWR?
+U 1 1 5C618B72
+P 2000 6750
+AR Path="/5C618B72" Ref="#PWR?"  Part="1"
+AR Path="/5C556B0F/5C618B72" Ref="#PWR0126"  Part="1"
+F 0 "#PWR0126" H 2000 6500 50  0001 C CNN
+F 1 "GND" H 2005 6577 50  0000 C CNN
+F 2 "" H 2000 6750 50  0001 C CNN
+F 3 "" H 2000 6750 50  0001 C CNN
+	1    2000 6750
+	1    0    0    -1
+$EndComp
+$Comp
+L power:+7.5V #PWR0129
+U 1 1 5C618BA1
+P 2000 6550
+F 0 "#PWR0129" H 2000 6400 50  0001 C CNN
+F 1 "+7.5V" V 2015 6678 50  0000 L CNN
+F 2 "" H 2000 6550 50  0001 C CNN
+F 3 "" H 2000 6550 50  0001 C CNN
+	1    2000 6550
+	0    -1   -1   0
+$EndComp
 $EndSCHEMATC
