File: HW/V2/SolderCon.sch (KiCad schematic (older format))
At the start: 17 parts, among them J1 WellerConn, Q1 Si4435, Q2 BSS138, Q3 Si4435, Q4 BSS138, U5 DS2401Z

Commit message: V2 milling and BOM
Other:
- note added: "Solders directly to MOSFET pins"
Changed lines of the file:
@@
 Wire Wire Line
 	3850 950  3800 950
+Text Notes 4800 1400 0    50   ~ 0
+Solders directly to MOSFET pins
 $EndSCHEMATC
